File: openbms/ADC.kicad_sch (KiCad schematic)
At the start: 117 parts, among them U1 DMP68D1LVQ-7, U10 DMP68D1LVQ-7, U11 DMN601VK-7, U12 DMN601VK-7, U13 DMN601VK-7, U14 DMN601VK-7, U2 DMP68D1LVQ-7, U3 DMN601VK-7, U4 DMP68D1LVQ-7, U5 ADS131M08xPBS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

Commit message: Capacitor values in ADC increased from 10n to 100n, production files released
Parts:
- C10, C11, C13, C15, C17, C18, C20: value 10n -> 100n; Manufacturer_Part_Number C0402C103K5REC7411 -> GRM155R71A104KA01D
- U5: Manufacturer_Part_Number (none) -> ADS131M08IPBS; Package (none) -> 32-TQFP
