File: openbms/Battery.kicad_sch (KiCad schematic)
At the start: 8 parts, among them J3 8-pin JST connector, J4 2-pin JST connector, J5 XT60PW-M connector

Commit message: Capacitor values in ADC increased from 10n to 100n, production files released
Parts:
- J4: Manufacturer_Parrt_Number S2B-XH-A -> (none); Manufacturer_Part_Number (none) -> S2B-XH-A; Package (none) -> 2-pin JST connector; Pakcage 2-pin JST connector -> (none)
- R104, R105, R106, R107, R114: now in the parts list
Changed lines of the file:
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@@
 		(unit 1)
 		(exclude_from_sim no)
-		(in_bom no)
+		(in_bom yes)
 		(on_board yes)
 		(dnp yes)
@@
 		)
 		(property "Manufacturer_Part_Number" "CR0402AJ/-000GAS"
+			(at 132.08 80.01 0)
+			(effects
+				(font
+					(size 1.27 1.27)
+				)
+				(hide yes)
+			)
+		)
+		(property "Pakcage" ""
 			(at 132.08 80.01 0)
 			(effects
@@
 		(unit 1)
 		(exclude_from_sim no)
-		(in_bom no)
+		(in_bom yes)
 		(on_board yes)
 		(dnp yes)
@@
 		)
 		(property "Manufacturer_Part_Number" "CR0402AJ/-000GAS"
+			(at 132.08 87.63 0)
+			(effects
+				(font
+					(size 1.27 1.27)
+				)
+				(hide yes)
+			)
+		)
+		(property "Pakcage" ""
 			(at 132.08 87.63 0)
 			(effects
@@
 		(unit 1)
 		(exclude_from_sim no)
-		(in_bom no)
+		(in_bom yes)
 		(on_board yes)
 		(dnp yes)
@@
 		)
 		(property "Manufacturer_Part_Number" "CR0402AJ/-000GAS"
+			(at 132.08 72.39 0)
+			(effects
+				(font
+					(size 1.27 1.27)
+				)
+				(hide yes)
+			)
+		)
+		(property "Pakcage" ""
 			(at 132.08 72.39 0)
 			(effects
@@
 		(unit 1)
 		(exclude_from_sim no)
-		(in_bom no)
+		(in_bom yes)
 		(on_board yes)
 		(dnp yes)
@@
 		)
 		(property "Manufacturer_Part_Number" "CR0402AJ/-000GAS"
+			(at 132.08 57.15 0)
+			(effects
+				(font
+					(size 1.27 1.27)
+				)
+				(hide yes)
+			)
+		)
+		(property "Pakcage" ""
 			(at 132.08 57.15 0)
 			(effects
@@
 		(unit 1)
 		(exclude_from_sim no)
-		(in_bom no)
+		(in_bom yes)
 		(on_board yes)
 		(dnp yes)
@@
 		)
 		(property "Manufacturer_Part_Number" "CR0402AJ/-000GAS"
+			(at 132.08 64.77 0)
+			(effects
+				(font
+					(size 1.27 1.27)
+				)
+				(hide yes)
+			)
+		)
+		(property "Pakcage" ""
 			(at 132.08 64.77 0)
 			(effects
@@
 			)
 		)
-		(property "Pakcage" "2-pin JST connector"
+		(property "Package" "2-pin JST connector"
 			(at 106.68 120.65 0)
 			(effects
@@
 			)
 		)
-		(property "Manufacturer_Parrt_Number" "S2B-XH-A"
+		(property "Manufacturer_Part_Number" "S2B-XH-A"
+			(at 106.68 120.65 0)
+			(effects
+				(font
+					(size 1.27 1.27)
+				)
+				(hide yes)
+			)
+		)
+		(property "Pakcage" ""
 			(at 106.68 120.65 0)
 			(effects
@@
 			)
 		)
+		(property "Pakcage" ""
+			(at 105.41 86.36 0)
+			(effects
+				(font
+					(size 1.27 1.27)
+				)
+				(hide yes)
+			)
+		)
 		(pin "4"
 		)
@@
 			(at 106.68 134.62 0)
 			(effects
+				(font
+					(size 1.27 1.27)
+				)
+				(hide yes)
+			)
+		)
+		(property "Pakcage" ""
+			(at 106.68 134.62 0)
+			(effects
