File: openbms/FETs.kicad_sch (KiCad schematic)
At the start: 29 parts, among them Q1 NTMFS5C612NLT1G, Q2 NTMFS5C612NLT1G, Q3 BSS84AKW,115, Q4 2N7002KW, Q5 2N7002KW, U18 DMP68D1LVQ-7, U19 TPS12000QDGXRQ1

Commit message: Capacitor values in ADC increased from 10n to 100n, production files released
Parts:
- Q1, Q2: Manufacturer_Part_Number (none) -> NTMFS5C612NLT1G
