File: openbms/MCU.kicad_sch (KiCad schematic)
At the start: 31 parts, among them J1 3-pin JST connector, J2 TagConnect_TC2030, U15 STM32L431CCUx, U16 TCAN3413DRBR, U17 32kbit EEPROM memory, Y2 8MHz

Commit message: Capacitor values in ADC increased from 10n to 100n, production files released
Parts:
- U15: Manufacturer_Part_Number (none) -> STM32L431CCU6TR; Package (none) -> 48-UFQFPN
