File: openbms/MCU.kicad_sch (KiCad schematic)
At the start: 31 parts, among them J1 3-pin JST connector, J2 TagConnect_TC2030, U15 STM32L431CCUx, U16 TCAN3413DRBR, U17 32kbit EEPROM memory, Y2 8MHz

Commit message: Footprints for pmos/nmos and pmos/pmos packages fixed, charger detection added, pwr_gd and flt_gd lines removed
Parts:
- added C35: 10n, Capacitor_SMD:C_0402_1005Metric, symbol Device:C_Small
- U15: footprint custom_library:QFN-48-1EP_7x7mm_P0.5mm_EP5.6x5.6mm -> Package_DFN_QFN:QFN-48-1EP_7x7mm_P0.5mm_EP5.6x5.6mm
- U16: footprint custom_library:SON65P300X300X100-9N-D -> custom_library:TCAN3413DRBR
Connections:
- net GND: now also C35.2; no longer U16.9 (EP)
- net BATT_NTC_POS renamed BATT_NTC_GND
- net BATT_NTC_GND: now also C35.1
- net DRV_FLT_GD renamed CHG_PRES
- net PWR_PG: no longer names the net of U15.20 (PB2)
Other:
- moved on the sheet: R86

Commit message: Option to shortcut current ADC sensor added
Connections:
- net CURR_CAL: now reaches U15.20 (PB2)
Changed lines of the file:
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@@
+		)
+	)
+	(hierarchical_label "CURR_CAL"
+		(shape output)
+		(at 142.24 127 180)
+		(effects
+			(font
+				(size 1.27 1.27)
+				(thickness 0.254)
+				(bold yes)
+				(color 0 0 132 1)
+			)
+			(justify right)
 		)
 	)

Commit message: Button for quick enable added
Parts:
- U15: footprint Package_DFN_QFN:QFN-48-1EP_7x7mm_P0.5mm_EP5.6x5.6mm -> custom_library:QFN-48-1EP_7x7mm_P0.5mm_EP5.6x5.6mm
Changed lines of the file:
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@@
 			)
 		)
-		(property "Footprint" "Package_DFN_QFN:QFN-48-1EP_7x7mm_P0.5mm_EP5.6x5.6mm"
+		(property "Footprint" "custom_library:QFN-48-1EP_7x7mm_P0.5mm_EP5.6x5.6mm"
 			(at 148.59 165.1 0)
 			(effects

Commit message: Green LED part number fixed,  PCB mask color updated, project description updated
Parts:
- D4: Manufacturer_Part_Number LTST-S270KGKT -> LTST-C190GKT
Changed lines of the file:
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@@
 	(title_block
 		(title "OpenBMS")
-		(date "2026-03-24")
-		(rev "A")
+		(date "2026-09-24")
+		(rev "B")
 		(comment 2 "More at openbatt.dev")
 		(comment 3 "Designed by OpenBatt team")
@@
 			)
 		)
-		(property "Manufacturer_Part_Number" "LTST-S270KGKT"
+		(property "Manufacturer_Part_Number" "LTST-C190GKT"
 			(at 262.89 93.98 0)
 			(effects

Commit message: Teardrops added, EEPROM part number updated, production files released
Parts:
- U17: Manufacturer_Part_Number M24C32-DRMN8TP/K -> M24256-DRMN8TP/K
Changed lines of the file:
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@@
 			)
 		)
-		(property "Manufacturer_Part_Number" "M24C32-DRMN8TP/K"
+		(property "Manufacturer_Part_Number" "M24256-DRMN8TP/K"
 			(at 158.75 218.44 0)
 			(effects

Commit message: BOM updates
Parts:
- U17: value 32kbit EEPROM memory -> 256kbit EEPROM memory
Changed lines of the file:
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@@
 			)
 		)
-		(property "Value" "32kbit EEPROM memory"
+		(property "Value" "256kbit EEPROM memory"
 			(at 161.544 225.552 0)
 			(effects
