File: openbms/openbms.kicad_pcb (KiCad board)
At the start: 4 copper layers, 68.4 x 52.4 mm, 210 parts, among them J1 3-pin JST connector, J2 TagConnect_TC2030, J3 8-pin JST connector, J4 2-pin JST connector, J5 XT60PW-M connector, J6 XT60PW-F connector, J7 7-pin JST connector, Q1 NTMFS5C612NLT1G, Q2 NTMFS5C612NLT1G, Q3 BSS84AKW,115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

Commit message: Capacitor values in ADC increased from 10n to 100n, production files released
Parts:
- C10, C11, C13, C15, C17, C18, C20: value 10n -> 100n
